File: hardware/heliopsis/heliopsis.sch (KiCad schematic (older format))
At the start: 10 parts, among them J1 NEIGHBOR1, J11 NEIGHBOR1, J12 NEIGHBOR2, J17 BONUS_ROW, J2 NEIGHBOR2, J7 BONUS_ROW

Commit message: Fix schematic component names (values)
Thanks @mossmann
Parts:
- J11: value NEIGHBOR1 -> NEIGHBOR11
- J12: value NEIGHBOR2 -> NEIGHBOR12
- J17: value BONUS_ROW -> BONUS_ROW1
Changed lines of the file:
@@
 P 12900 2600
 F 0 "J12" H 12900 3650 50  0000 C CNN
-F 1 "NEIGHBOR2" V 12900 2600 50  0000 C CNN
+F 1 "NEIGHBOR12" V 12900 2600 50  0000 C CNN
 F 2 "gsg-modules:HEADER-2x20" H 12900 1650 60  0001 C CNN
 F 3 "" H 12900 1650 60  0000 C CNN
@@
 P 12900 5200
 F 0 "J11" H 12900 6250 50  0000 C CNN
-F 1 "NEIGHBOR1" V 12900 5200 50  0000 C CNN
+F 1 "NEIGHBOR11" V 12900 5200 50  0000 C CNN
 F 2 "gsg-modules:HEADER-2x20" H 12900 4250 60  0001 C CNN
 F 3 "" H 12900 4250 60  0000 C CNN
@@
 P 12350 6950
 F 0 "J17" H 12350 8000 50  0000 C CNN
-F 1 "BONUS_ROW" V 12450 6950 50  0000 C CNN
+F 1 "BONUS_ROW1" V 12450 6950 50  0000 C CNN
 F 2 "gsg-modules:HEADER-1x20" H 12350 6950 60  0001 C CNN
 F 3 "" H 12350 6950 60  0000 C CNN
