File: hardware/heliopsis/heliopsis.kicad_pcb (KiCad board)
At the start: 2 copper layers, 70.7 x 53.3 mm, 10 parts, among them J1 NEIGHBOR1, J11 NEIGHBOR1, J12 NEIGHBOR2, J17 BONUS_ROW, J2 NEIGHBOR2, J7 BONUS_ROW

Commit message: Add SMD pad to board
Parts:
- added P1: smd-proto-pad-hole, heliopsis-modules:smd-proto-pad-hole, F.Cu at (171.4, 88.9)
Changed lines of the file:
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@@
 (kicad_pcb (version 4) (host pcbnew 4.0.2-stable)
   (general
-    (links 141)
-    (no_connects 0)
+    (links 0)
+    (no_connects 1)
     (area 107.95 66.04 279.525801 124.460001)
     (thickness 1.6)
@@
     (tracks 369)
     (zones 0)
-    (modules 10)
+    (modules 11)
     (nets 96)
   )
@@
   )
   (setup
-    (last_trace_width 0.2032)
+    (last_trace_width 0.3048)
     (user_trace_width 0.3048)
     (user_trace_width 0.508)
@@
       (net 2 VCC))
   )
+  (module heliopsis-modules:smd-proto-pad-hole (layer F.Cu)
+    (at 171.45 88.9)
+    (descr "SMD prototyping pad with unplated hole to bottom side for optional ground plane (or other signal)")
+    (attr virtual)
+    (fp_text reference P1 (at 0 3.04) (layer F.SilkS) hide
+      (effects (font (size 1 1) (thickness 0.15)))
+    )
+    (fp_text value smd-proto-pad-hole (at 0 2.04) (layer F.Fab) hide
+      (effects (font (size 1 1) (thickness 0.15)))
+    )
+    (pad 1 connect rect (at 0 0) (size 1.2954 0.9144) (layers F.Cu F.Mask))
+    (pad 2 connect rect (at 0 0) (size 1.2954 0.9144) (layers B.Cu B.Mask)
+      (net 1 GND))
+    (pad "" np_thru_hole circle (at 0 0) (size 0.762 0.762) (drill 0.762) (layers *.Cu *.Mask))
+  )
   (gr_line (start 109.6772 98.933) (end 109.728 99.9998) (angle 90) (layer Edge.Cuts) (width 0.15))

Commit message: Redesign SMD prototyping pad
The original design for pad with a nonplated hole to optionally connect
to a ground plane does not seem to be easily designed.
Parts:
- removed P1: smd-proto-pad-hole, heliopsis-modules:smd-proto-pad-hole
Changed lines of the file:
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@@
 (kicad_pcb (version 4) (host pcbnew 4.0.2-stable)
   (general
-    (links 0)
-    (no_connects 1)
+    (links 141)
+    (no_connects 0)
     (area 107.95 66.04 279.525801 124.460001)
     (thickness 1.6)
@@
     (tracks 369)
     (zones 0)
-    (modules 11)
+    (modules 10)
     (nets 96)
   )
@@
   )
   (setup
-    (last_trace_width 0.3048)
+    (last_trace_width 0.2032)
     (user_trace_width 0.3048)
     (user_trace_width 0.508)
@@
       (net 2 VCC))
   )
-  (module heliopsis-modules:smd-proto-pad-hole (layer F.Cu)
-    (at 171.45 88.9)
-    (descr "SMD prototyping pad with unplated hole to bottom side for optional ground plane (or other signal)")
-    (attr virtual)
-    (fp_text reference P1 (at 0 3.04) (layer F.SilkS) hide
-      (effects (font (size 1 1) (thickness 0.15)))
-    )
-    (fp_text value smd-proto-pad-hole (at 0 2.04) (layer F.Fab) hide
-      (effects (font (size 1 1) (thickness 0.15)))
-    )
-    (pad 1 connect rect (at 0 0) (size 1.2954 0.9144) (layers F.Cu F.Mask))
-    (pad 2 connect rect (at 0 0) (size 1.2954 0.9144) (layers B.Cu B.Mask)
-      (net 1 GND))
-    (pad "" np_thru_hole circle (at 0 0) (size 0.762 0.762) (drill 0.762) (layers *.Cu *.Mask))
-  )
   (gr_line (start 109.6772 98.933) (end 109.728 99.9998) (angle 90) (layer Edge.Cuts) (width 0.15))

Commit message: Add SMD and PTH photo (autoincorrect) areas!
Parts:
- added P1101: smd-proto-pad, heliopsis-modules:smd-proto-pad, F.Cu at (156.6, 88.9)
- added P11010: smd-proto-pad, heliopsis-modules:smd-proto-pad, F.Cu at (156.6, 100.3)
- added P11011: smd-proto-pad, heliopsis-modules:smd-proto-pad, F.Cu at (156.6, 101.6)
- added P11012: smd-proto-pad, heliopsis-modules:smd-proto-pad, F.Cu at (156.6, 102.9)
- added P11013: smd-proto-pad, heliopsis-modules:smd-proto-pad, F.Cu at (156.6, 104.1)
- added P11014: smd-proto-pad, heliopsis-modules:smd-proto-pad, F.Cu at (156.6, 105.4)
- added P11015: smd-proto-pad, heliopsis-modules:smd-proto-pad, F.Cu at (156.6, 106.7)
- added P1102: smd-proto-pad, heliopsis-modules:smd-proto-pad, F.Cu at (156.6, 90.2)
- added P1103: smd-proto-pad, heliopsis-modules:smd-proto-pad, F.Cu at (156.6, 91.4)
- added P1104: smd-proto-pad, heliopsis-modules:smd-proto-pad, F.Cu at (156.6, 92.7)
- added P1105: smd-proto-pad, heliopsis-modules:smd-proto-pad, F.Cu at (156.6, 94.0)
- added P1106: smd-proto-pad, heliopsis-modules:smd-proto-pad, F.Cu at (156.6, 95.2)
- added P1107: smd-proto-pad, heliopsis-modules:smd-proto-pad, F.Cu at (156.6, 96.5)
- added P1108: smd-proto-pad, heliopsis-modules:smd-proto-pad, F.Cu at (156.6, 97.8)
- added P1109: smd-proto-pad, heliopsis-modules:smd-proto-pad, F.Cu at (156.6, 99.1)
- added P111: smd-proto-pad, heliopsis-modules:smd-proto-pad, F.Cu at (171.4, 88.9)
- added P1110: smd-proto-pad, heliopsis-modules:smd-proto-pad, F.Cu at (171.4, 100.3)
- added P1111: smd-proto-pad, heliopsis-modules:smd-proto-pad, F.Cu at (171.4, 101.6)
- added P1111: smd-proto-pad, heliopsis-modules:smd-proto-pad, F.Cu at (154.9, 88.9)
- added P11110: smd-proto-pad, heliopsis-modules:smd-proto-pad, F.Cu at (154.9, 100.3)
- added P11111: smd-proto-pad, heliopsis-modules:smd-proto-pad, F.Cu at (154.9, 101.6)
- added P11112: smd-proto-pad, heliopsis-modules:smd-proto-pad, F.Cu at (154.9, 102.9)
- added P11113: smd-proto-pad, heliopsis-modules:smd-proto-pad, F.Cu at (154.9, 104.1)
- added P11114: smd-proto-pad, heliopsis-modules:smd-proto-pad, F.Cu at (154.9, 105.4)
- added P11115: smd-proto-pad, heliopsis-modules:smd-proto-pad, F.Cu at (154.9, 106.7)
- added P1112: smd-proto-pad, heliopsis-modules:smd-proto-pad, F.Cu at (171.4, 102.9)
- added P1112: smd-proto-pad, heliopsis-modules:smd-proto-pad, F.Cu at (154.9, 90.2)
- added P1113: smd-proto-pad, heliopsis-modules:smd-proto-pad, F.Cu at (171.4, 104.1)
- added P1113: smd-proto-pad, heliopsis-modules:smd-proto-pad, F.Cu at (154.9, 91.4)
- added P1114: smd-proto-pad, heliopsis-modules:smd-proto-pad, F.Cu at (171.4, 105.4)
- added P1114: smd-proto-pad, heliopsis-modules:smd-proto-pad, F.Cu at (154.9, 92.7)
- added P1115: smd-proto-pad, heliopsis-modules:smd-proto-pad, F.Cu at (171.4, 106.7)
- added P1115: smd-proto-pad, heliopsis-modules:smd-proto-pad, F.Cu at (154.9, 94.0)
- added P1116: smd-proto-pad, heliopsis-modules:smd-proto-pad, F.Cu at (154.9, 95.2)
- added P1117: smd-proto-pad, heliopsis-modules:smd-proto-pad, F.Cu at (154.9, 96.5)
- added P1118: smd-proto-pad, heliopsis-modules:smd-proto-pad, F.Cu at (154.9, 97.8)
- added P1119: smd-proto-pad, heliopsis-modules:smd-proto-pad, F.Cu at (154.9, 99.1)
- added P112: smd-proto-pad, heliopsis-modules:smd-proto-pad, F.Cu at (171.4, 90.2)
- added P1121: smd-proto-pad, heliopsis-modules:smd-proto-pad, F.Cu at (153.3, 88.9)
- added P11210: smd-proto-pad, heliopsis-modules:smd-proto-pad, F.Cu at (153.3, 100.3)
- added P11211: smd-proto-pad, heliopsis-modules:smd-proto-pad, F.Cu at (153.3, 101.6)
- added P11212: smd-proto-pad, heliopsis-modules:smd-proto-pad, F.Cu at (153.3, 102.9)
- added P11213: smd-proto-pad, heliopsis-modules:smd-proto-pad, F.Cu at (153.3, 104.1)
- added P11214: smd-proto-pad, heliopsis-modules:smd-proto-pad, F.Cu at (153.3, 105.4)
- added P11215: smd-proto-pad, heliopsis-modules:smd-proto-pad, F.Cu at (153.3, 106.7)
- added P1122: smd-proto-pad, heliopsis-modules:smd-proto-pad, F.Cu at (153.3, 90.2)
- added P1123: smd-proto-pad, heliopsis-modules:smd-proto-pad, F.Cu at (153.3, 91.4)
- added P1124: smd-proto-pad, heliopsis-modules:smd-proto-pad, F.Cu at (153.3, 92.7)
- added P1125: smd-proto-pad, heliopsis-modules:smd-proto-pad, F.Cu at (153.3, 94.0)
- added P1126: smd-proto-pad, heliopsis-modules:smd-proto-pad, F.Cu at (153.3, 95.2)
- added P1127: smd-proto-pad, heliopsis-modules:smd-proto-pad, F.Cu at (153.3, 96.5)
- added P1128: smd-proto-pad, heliopsis-modules:smd-proto-pad, F.Cu at (153.3, 97.8)
- added P1129: smd-proto-pad, heliopsis-modules:smd-proto-pad, F.Cu at (153.3, 99.1)
- added P113: smd-proto-pad, heliopsis-modules:smd-proto-pad, F.Cu at (171.4, 91.4)
- added P1131: smd-proto-pad, heliopsis-modules:smd-proto-pad, F.Cu at (151.6, 88.9)
- added P11310: smd-proto-pad, heliopsis-modules:smd-proto-pad, F.Cu at (151.6, 100.3)
- added P11311: smd-proto-pad, heliopsis-modules:smd-proto-pad, F.Cu at (151.6, 101.6)
- added P11312: smd-proto-pad, heliopsis-modules:smd-proto-pad, F.Cu at (151.6, 102.9)
- added P11313: smd-proto-pad, heliopsis-modules:smd-proto-pad, F.Cu at (151.6, 104.1)
- added P11314: smd-proto-pad, heliopsis-modules:smd-proto-pad, F.Cu at (151.6, 105.4)
- added P11315: smd-proto-pad, heliopsis-modules:smd-proto-pad, F.Cu at (151.6, 106.7)
- added P1132: smd-proto-pad, heliopsis-modules:smd-proto-pad, F.Cu at (151.6, 90.2)
- added P1133: smd-proto-pad, heliopsis-modules:smd-proto-pad, F.Cu at (151.6, 91.4)
- added P1134: smd-proto-pad, heliopsis-modules:smd-proto-pad, F.Cu at (151.6, 92.7)
- added P1135: smd-proto-pad, heliopsis-modules:smd-proto-pad, F.Cu at (151.6, 94.0)
- added P1136: smd-proto-pad, heliopsis-modules:smd-proto-pad, F.Cu at (151.6, 95.2)
- added P1137: smd-proto-pad, heliopsis-modules:smd-proto-pad, F.Cu at (151.6, 96.5)
- added P1138: smd-proto-pad, heliopsis-modules:smd-proto-pad, F.Cu at (151.6, 97.8)
- added P1139: smd-proto-pad, heliopsis-modules:smd-proto-pad, F.Cu at (151.6, 99.1)
- added P114: smd-proto-pad, heliopsis-modules:smd-proto-pad, F.Cu at (171.4, 92.7)
- added P1141: smd-proto-pad, heliopsis-modules:smd-proto-pad, F.Cu at (150.0, 88.9)
- added P11410: smd-proto-pad, heliopsis-modules:smd-proto-pad, F.Cu at (150.0, 100.3)
- added P11411: smd-proto-pad, heliopsis-modules:smd-proto-pad, F.Cu at (150.0, 101.6)
- added P11412: smd-proto-pad, heliopsis-modules:smd-proto-pad, F.Cu at (150.0, 102.9)
- added P11413: smd-proto-pad, heliopsis-modules:smd-proto-pad, F.Cu at (150.0, 104.1)
- added P11414: smd-proto-pad, heliopsis-modules:smd-proto-pad, F.Cu at (150.0, 105.4)
- added P11415: smd-proto-pad, heliopsis-modules:smd-proto-pad, F.Cu at (150.0, 106.7)
- added P1142: smd-proto-pad, heliopsis-modules:smd-proto-pad, F.Cu at (150.0, 90.2)
- added P1143: smd-proto-pad, heliopsis-modules:smd-proto-pad, F.Cu at (150.0, 91.4)
- added P1144: smd-proto-pad, heliopsis-modules:smd-proto-pad, F.Cu at (150.0, 92.7)
- added P1145: smd-proto-pad, heliopsis-modules:smd-proto-pad, F.Cu at (150.0, 94.0)
- added P1146: smd-proto-pad, heliopsis-modules:smd-proto-pad, F.Cu at (150.0, 95.2)
- added P1147: smd-proto-pad, heliopsis-modules:smd-proto-pad, F.Cu at (150.0, 96.5)
- added P1148: smd-proto-pad, heliopsis-modules:smd-proto-pad, F.Cu at (150.0, 97.8)
- added P1149: smd-proto-pad, heliopsis-modules:smd-proto-pad, F.Cu at (150.0, 99.1)
- added P115: smd-proto-pad, heliopsis-modules:smd-proto-pad, F.Cu at (171.4, 94.0)
- added P1151: smd-proto-pad, heliopsis-modules:smd-proto-pad, F.Cu at (148.3, 88.9)
- added P11510: smd-proto-pad, heliopsis-modules:smd-proto-pad, F.Cu at (148.3, 100.3)
- added P11511: smd-proto-pad, heliopsis-modules:smd-proto-pad, F.Cu at (148.3, 101.6)
- added P11512: smd-proto-pad, heliopsis-modules:smd-proto-pad, F.Cu at (148.3, 102.9)
- added P11513: smd-proto-pad, heliopsis-modules:smd-proto-pad, F.Cu at (148.3, 104.1)
- added P11514: smd-proto-pad, heliopsis-modules:smd-proto-pad, F.Cu at (148.3, 105.4)
- added P11515: smd-proto-pad, heliopsis-modules:smd-proto-pad, F.Cu at (148.3, 106.7)
- added P1152: smd-proto-pad, heliopsis-modules:smd-proto-pad, F.Cu at (148.3, 90.2)
- added P1153: smd-proto-pad, heliopsis-modules:smd-proto-pad, F.Cu at (148.3, 91.4)
- added P1154: smd-proto-pad, heliopsis-modules:smd-proto-pad, F.Cu at (148.3, 92.7)
- added P1155: smd-proto-pad, heliopsis-modules:smd-proto-pad, F.Cu at (148.3, 94.0)
- added P1156: smd-proto-pad, heliopsis-modules:smd-proto-pad, F.Cu at (148.3, 95.2)
- added P1157: smd-proto-pad, heliopsis-modules:smd-proto-pad, F.Cu at (148.3, 96.5)
- added P1158: smd-proto-pad, heliopsis-modules:smd-proto-pad, F.Cu at (148.3, 97.8)
- added P1159: smd-proto-pad, heliopsis-modules:smd-proto-pad, F.Cu at (148.3, 99.1)
- added P116: smd-proto-pad, heliopsis-modules:smd-proto-pad, F.Cu at (171.4, 95.2)
- added P1161: smd-proto-pad, heliopsis-modules:smd-proto-pad, F.Cu at (146.7, 88.9)
- added P11610: smd-proto-pad, heliopsis-modules:smd-proto-pad, F.Cu at (146.7, 100.3)
- added P11611: smd-proto-pad, heliopsis-modules:smd-proto-pad, F.Cu at (146.7, 101.6)
- added P11612: smd-proto-pad, heliopsis-modules:smd-proto-pad, F.Cu at (146.7, 102.9)
- added P11613: smd-proto-pad, heliopsis-modules:smd-proto-pad, F.Cu at (146.7, 104.1)
- added P11614: smd-proto-pad, heliopsis-modules:smd-proto-pad, F.Cu at (146.7, 105.4)
- added P11615: smd-proto-pad, heliopsis-modules:smd-proto-pad, F.Cu at (146.7, 106.7)
- added P1162: smd-proto-pad, heliopsis-modules:smd-proto-pad, F.Cu at (146.7, 90.2)
- added P1163: smd-proto-pad, heliopsis-modules:smd-proto-pad, F.Cu at (146.7, 91.4)
- added P1164: smd-proto-pad, heliopsis-modules:smd-proto-pad, F.Cu at (146.7, 92.7)
- added P1165: smd-proto-pad, heliopsis-modules:smd-proto-pad, F.Cu at (146.7, 94.0)
- added P1166: smd-proto-pad, heliopsis-modules:smd-proto-pad, F.Cu at (146.7, 95.2)
- added P1167: smd-proto-pad, heliopsis-modules:smd-proto-pad, F.Cu at (146.7, 96.5)
- added P1168: smd-proto-pad, heliopsis-modules:smd-proto-pad, F.Cu at (146.7, 97.8)
- added P1169: smd-proto-pad, heliopsis-modules:smd-proto-pad, F.Cu at (146.7, 99.1)
- added P117: smd-proto-pad, heliopsis-modules:smd-proto-pad, F.Cu at (171.4, 96.5)
- added P1171: smd-proto-pad, heliopsis-modules:smd-proto-pad, F.Cu at (145.0, 88.9)
- added P11710: smd-proto-pad, heliopsis-modules:smd-proto-pad, F.Cu at (145.0, 100.3)
- added P11711: smd-proto-pad, heliopsis-modules:smd-proto-pad, F.Cu at (145.0, 101.6)
- added P11712: smd-proto-pad, heliopsis-modules:smd-proto-pad, F.Cu at (145.0, 102.9)
- added P11713: smd-proto-pad, heliopsis-modules:smd-proto-pad, F.Cu at (145.0, 104.1)
- added P11714: smd-proto-pad, heliopsis-modules:smd-proto-pad, F.Cu at (145.0, 105.4)
- added P11715: smd-proto-pad, heliopsis-modules:smd-proto-pad, F.Cu at (145.0, 106.7)
- added P1172: smd-proto-pad, heliopsis-modules:smd-proto-pad, F.Cu at (145.0, 90.2)
- added P1173: smd-proto-pad, heliopsis-modules:smd-proto-pad, F.Cu at (145.0, 91.4)
- added P1174: smd-proto-pad, heliopsis-modules:smd-proto-pad, F.Cu at (145.0, 92.7)
- added P1175: smd-proto-pad, heliopsis-modules:smd-proto-pad, F.Cu at (145.0, 94.0)
- added P1176: smd-proto-pad, heliopsis-modules:smd-proto-pad, F.Cu at (145.0, 95.2)
- added P1177: smd-proto-pad, heliopsis-modules:smd-proto-pad, F.Cu at (145.0, 96.5)
- added P1178: smd-proto-pad, heliopsis-modules:smd-proto-pad, F.Cu at (145.0, 97.8)
- added P1179: smd-proto-pad, heliopsis-modules:smd-proto-pad, F.Cu at (145.0, 99.1)
- added P118: smd-proto-pad, heliopsis-modules:smd-proto-pad, F.Cu at (171.4, 97.8)
- added P1181: smd-proto-pad, heliopsis-modules:smd-proto-pad, F.Cu at (143.4, 88.9)
- added P11810: smd-proto-pad, heliopsis-modules:smd-proto-pad, F.Cu at (143.4, 100.3)
- added P11811: smd-proto-pad, heliopsis-modules:smd-proto-pad, F.Cu at (143.4, 101.6)
- added P11812: smd-proto-pad, heliopsis-modules:smd-proto-pad, F.Cu at (143.4, 102.9)
- added P11813: smd-proto-pad, heliopsis-modules:smd-proto-pad, F.Cu at (143.4, 104.1)
- added P11814: smd-proto-pad, heliopsis-modules:smd-proto-pad, F.Cu at (143.4, 105.4)
- added P11815: smd-proto-pad, heliopsis-modules:smd-proto-pad, F.Cu at (143.4, 106.7)
- added P1182: smd-proto-pad, heliopsis-modules:smd-proto-pad, F.Cu at (143.4, 90.2)
- added P1183: smd-proto-pad, heliopsis-modules:smd-proto-pad, F.Cu at (143.4, 91.4)
- added P1184: smd-proto-pad, heliopsis-modules:smd-proto-pad, F.Cu at (143.4, 92.7)
- added P1185: smd-proto-pad, heliopsis-modules:smd-proto-pad, F.Cu at (143.4, 94.0)
- added P1186: smd-proto-pad, heliopsis-modules:smd-proto-pad, F.Cu at (143.4, 95.2)
- added P1187: smd-proto-pad, heliopsis-modules:smd-proto-pad, F.Cu at (143.4, 96.5)
- added P1188: smd-proto-pad, heliopsis-modules:smd-proto-pad, F.Cu at (143.4, 97.8)
- added P1189: smd-proto-pad, heliopsis-modules:smd-proto-pad, F.Cu at (143.4, 99.1)
- added P119: smd-proto-pad, heliopsis-modules:smd-proto-pad, F.Cu at (171.4, 99.1)
- added P1191: smd-proto-pad, heliopsis-modules:smd-proto-pad, F.Cu at (141.7, 88.9)
- added P11910: smd-proto-pad, heliopsis-modules:smd-proto-pad, F.Cu at (141.7, 100.3)
- added P11911: smd-proto-pad, heliopsis-modules:smd-proto-pad, F.Cu at (141.7, 101.6)
- added P11912: smd-proto-pad, heliopsis-modules:smd-proto-pad, F.Cu at (141.7, 102.9)
- added P11913: smd-proto-pad, heliopsis-modules:smd-proto-pad, F.Cu at (141.7, 104.1)
- added P11914: smd-proto-pad, heliopsis-modules:smd-proto-pad, F.Cu at (141.7, 105.4)
- added P11915: smd-proto-pad, heliopsis-modules:smd-proto-pad, F.Cu at (141.7, 106.7)
- added P1192: smd-proto-pad, heliopsis-modules:smd-proto-pad, F.Cu at (141.7, 90.2)
- added P1193: smd-proto-pad, heliopsis-modules:smd-proto-pad, F.Cu at (141.7, 91.4)
- added P1194: smd-proto-pad, heliopsis-modules:smd-proto-pad, F.Cu at (141.7, 92.7)
- added P1195: smd-proto-pad, heliopsis-modules:smd-proto-pad, F.Cu at (141.7, 94.0)
- added P1196: smd-proto-pad, heliopsis-modules:smd-proto-pad, F.Cu at (141.7, 95.2)
- added P1197: smd-proto-pad, heliopsis-modules:smd-proto-pad, F.Cu at (141.7, 96.5)
- added P1198: smd-proto-pad, heliopsis-modules:smd-proto-pad, F.Cu at (141.7, 97.8)
- added P1199: smd-proto-pad, heliopsis-modules:smd-proto-pad, F.Cu at (141.7, 99.1)
- added P1201: smd-proto-pad, heliopsis-modules:smd-proto-pad, F.Cu at (140.1, 88.9)
- added P12010: smd-proto-pad, heliopsis-modules:smd-proto-pad, F.Cu at (140.1, 100.3)
- added P12011: smd-proto-pad, heliopsis-modules:smd-proto-pad, F.Cu at (140.1, 101.6)
- added P12012: smd-proto-pad, heliopsis-modules:smd-proto-pad, F.Cu at (140.1, 102.9)
- added P12013: smd-proto-pad, heliopsis-modules:smd-proto-pad, F.Cu at (140.1, 104.1)
- added P12014: smd-proto-pad, heliopsis-modules:smd-proto-pad, F.Cu at (140.1, 105.4)
- added P12015: smd-proto-pad, heliopsis-modules:smd-proto-pad, F.Cu at (140.1, 106.7)
- added P1202: smd-proto-pad, heliopsis-modules:smd-proto-pad, F.Cu at (140.1, 90.2)
- added P1203: smd-proto-pad, heliopsis-modules:smd-proto-pad, F.Cu at (140.1, 91.4)
- added P1204: smd-proto-pad, heliopsis-modules:smd-proto-pad, F.Cu at (140.1, 92.7)
- added P1205: smd-proto-pad, heliopsis-modules:smd-proto-pad, F.Cu at (140.1, 94.0)
- added P1206: smd-proto-pad, heliopsis-modules:smd-proto-pad, F.Cu at (140.1, 95.2)
- added P1207: smd-proto-pad, heliopsis-modules:smd-proto-pad, F.Cu at (140.1, 96.5)
- added P1208: smd-proto-pad, heliopsis-modules:smd-proto-pad, F.Cu at (140.1, 97.8)
- added P1209: smd-proto-pad, heliopsis-modules:smd-proto-pad, F.Cu at (140.1, 99.1)
- added P121: smd-proto-pad, heliopsis-modules:smd-proto-pad, F.Cu at (169.8, 88.9)
- added P1210: smd-proto-pad, heliopsis-modules:smd-proto-pad, F.Cu at (169.8, 100.3)
- added P1211: smd-proto-pad, heliopsis-modules:smd-proto-pad, F.Cu at (169.8, 101.6)
- added P1212: smd-proto-pad, heliopsis-modules:smd-proto-pad, F.Cu at (169.8, 102.9)
- added P1213: smd-proto-pad, heliopsis-modules:smd-proto-pad, F.Cu at (169.8, 104.1)
- added P1214: smd-proto-pad, heliopsis-modules:smd-proto-pad, F.Cu at (169.8, 105.4)
- added P1215: smd-proto-pad, heliopsis-modules:smd-proto-pad, F.Cu at (169.8, 106.7)
- added P122: smd-proto-pad, heliopsis-modules:smd-proto-pad, F.Cu at (169.8, 90.2)
- added P123: smd-proto-pad, heliopsis-modules:smd-proto-pad, F.Cu at (169.8, 91.4)
- added P124: smd-proto-pad, heliopsis-modules:smd-proto-pad, F.Cu at (169.8, 92.7)
- added P125: smd-proto-pad, heliopsis-modules:smd-proto-pad, F.Cu at (169.8, 94.0)
- added P126: smd-proto-pad, heliopsis-modules:smd-proto-pad, F.Cu at (169.8, 95.2)
- added P127: smd-proto-pad, heliopsis-modules:smd-proto-pad, F.Cu at (169.8, 96.5)
- added P128: smd-proto-pad, heliopsis-modules:smd-proto-pad, F.Cu at (169.8, 97.8)
- added P129: smd-proto-pad, heliopsis-modules:smd-proto-pad, F.Cu at (169.8, 99.1)
- added P131: smd-proto-pad, heliopsis-modules:smd-proto-pad, F.Cu at (168.1, 88.9)
- added P1310: smd-proto-pad, heliopsis-modules:smd-proto-pad, F.Cu at (168.1, 100.3)
- added P1311: smd-proto-pad, heliopsis-modules:smd-proto-pad, F.Cu at (168.1, 101.6)
- added P1312: smd-proto-pad, heliopsis-modules:smd-proto-pad, F.Cu at (168.1, 102.9)
- added P1313: smd-proto-pad, heliopsis-modules:smd-proto-pad, F.Cu at (168.1, 104.1)
- added P1314: smd-proto-pad, heliopsis-modules:smd-proto-pad, F.Cu at (168.1, 105.4)
- added P1315: smd-proto-pad, heliopsis-modules:smd-proto-pad, F.Cu at (168.1, 106.7)
- added P132: smd-proto-pad, heliopsis-modules:smd-proto-pad, F.Cu at (168.1, 90.2)
- added P133: smd-proto-pad, heliopsis-modules:smd-proto-pad, F.Cu at (168.1, 91.4)
- added P134: smd-proto-pad, heliopsis-modules:smd-proto-pad, F.Cu at (168.1, 92.7)
- added P135: smd-proto-pad, heliopsis-modules:smd-proto-pad, F.Cu at (168.1, 94.0)
- added P136: smd-proto-pad, heliopsis-modules:smd-proto-pad, F.Cu at (168.1, 95.2)
- added P137: smd-proto-pad, heliopsis-modules:smd-proto-pad, F.Cu at (168.1, 96.5)
- added P138: smd-proto-pad, heliopsis-modules:smd-proto-pad, F.Cu at (168.1, 97.8)
- added P139: smd-proto-pad, heliopsis-modules:smd-proto-pad, F.Cu at (168.1, 99.1)
- added P141: smd-proto-pad, heliopsis-modules:smd-proto-pad, F.Cu at (166.5, 88.9)
- added P1410: smd-proto-pad, heliopsis-modules:smd-proto-pad, F.Cu at (166.5, 100.3)
- added P1411: smd-proto-pad, heliopsis-modules:smd-proto-pad, F.Cu at (166.5, 101.6)
- added P1412: smd-proto-pad, heliopsis-modules:smd-proto-pad, F.Cu at (166.5, 102.9)
- added P1413: smd-proto-pad, heliopsis-modules:smd-proto-pad, F.Cu at (166.5, 104.1)
- added P1414: smd-proto-pad, heliopsis-modules:smd-proto-pad, F.Cu at (166.5, 105.4)
- added P1415: smd-proto-pad, heliopsis-modules:smd-proto-pad, F.Cu at (166.5, 106.7)
- added P142: smd-proto-pad, heliopsis-modules:smd-proto-pad, F.Cu at (166.5, 90.2)
- added P143: smd-proto-pad, heliopsis-modules:smd-proto-pad, F.Cu at (166.5, 91.4)
- added P144: smd-proto-pad, heliopsis-modules:smd-proto-pad, F.Cu at (166.5, 92.7)
- added P145: smd-proto-pad, heliopsis-modules:smd-proto-pad, F.Cu at (166.5, 94.0)
- added P146: smd-proto-pad, heliopsis-modules:smd-proto-pad, F.Cu at (166.5, 95.2)
- added P147: smd-proto-pad, heliopsis-modules:smd-proto-pad, F.Cu at (166.5, 96.5)
- added P148: smd-proto-pad, heliopsis-modules:smd-proto-pad, F.Cu at (166.5, 97.8)
- added P149: smd-proto-pad, heliopsis-modules:smd-proto-pad, F.Cu at (166.5, 99.1)
- added P151: smd-proto-pad, heliopsis-modules:smd-proto-pad, F.Cu at (164.8, 88.9)
- added P1510: smd-proto-pad, heliopsis-modules:smd-proto-pad, F.Cu at (164.8, 100.3)
- added P1511: smd-proto-pad, heliopsis-modules:smd-proto-pad, F.Cu at (164.8, 101.6)
- added P1512: smd-proto-pad, heliopsis-modules:smd-proto-pad, F.Cu at (164.8, 102.9)
- added P1513: smd-proto-pad, heliopsis-modules:smd-proto-pad, F.Cu at (164.8, 104.1)
- added P1514: smd-proto-pad, heliopsis-modules:smd-proto-pad, F.Cu at (164.8, 105.4)
- added P1515: smd-proto-pad, heliopsis-modules:smd-proto-pad, F.Cu at (164.8, 106.7)
- added P152: smd-proto-pad, heliopsis-modules:smd-proto-pad, F.Cu at (164.8, 90.2)
- added P153: smd-proto-pad, heliopsis-modules:smd-proto-pad, F.Cu at (164.8, 91.4)
- added P154: smd-proto-pad, heliopsis-modules:smd-proto-pad, F.Cu at (164.8, 92.7)
- added P155: smd-proto-pad, heliopsis-modules:smd-proto-pad, F.Cu at (164.8, 94.0)
- added P156: smd-proto-pad, heliopsis-modules:smd-proto-pad, F.Cu at (164.8, 95.2)
- added P157: smd-proto-pad, heliopsis-modules:smd-proto-pad, F.Cu at (164.8, 96.5)
- added P158: smd-proto-pad, heliopsis-modules:smd-proto-pad, F.Cu at (164.8, 97.8)
- added P159: smd-proto-pad, heliopsis-modules:smd-proto-pad, F.Cu at (164.8, 99.1)
- added P161: smd-proto-pad, heliopsis-modules:smd-proto-pad, F.Cu at (163.2, 88.9)
- added P1610: smd-proto-pad, heliopsis-modules:smd-proto-pad, F.Cu at (163.2, 100.3)
- added P1611: smd-proto-pad, heliopsis-modules:smd-proto-pad, F.Cu at (163.2, 101.6)
- added P1612: smd-proto-pad, heliopsis-modules:smd-proto-pad, F.Cu at (163.2, 102.9)
- added P1613: smd-proto-pad, heliopsis-modules:smd-proto-pad, F.Cu at (163.2, 104.1)
- added P1614: smd-proto-pad, heliopsis-modules:smd-proto-pad, F.Cu at (163.2, 105.4)
- added P1615: smd-proto-pad, heliopsis-modules:smd-proto-pad, F.Cu at (163.2, 106.7)
- added P162: smd-proto-pad, heliopsis-modules:smd-proto-pad, F.Cu at (163.2, 90.2)
- added P163: smd-proto-pad, heliopsis-modules:smd-proto-pad, F.Cu at (163.2, 91.4)
- added P164: smd-proto-pad, heliopsis-modules:smd-proto-pad, F.Cu at (163.2, 92.7)
- added P165: smd-proto-pad, heliopsis-modules:smd-proto-pad, F.Cu at (163.2, 94.0)
- added P166: smd-proto-pad, heliopsis-modules:smd-proto-pad, F.Cu at (163.2, 95.2)
- added P167: smd-proto-pad, heliopsis-modules:smd-proto-pad, F.Cu at (163.2, 96.5)
- added P168: smd-proto-pad, heliopsis-modules:smd-proto-pad, F.Cu at (163.2, 97.8)
- added P169: smd-proto-pad, heliopsis-modules:smd-proto-pad, F.Cu at (163.2, 99.1)
- added P171: smd-proto-pad, heliopsis-modules:smd-proto-pad, F.Cu at (161.5, 88.9)
- added P1710: smd-proto-pad, heliopsis-modules:smd-proto-pad, F.Cu at (161.5, 100.3)
- added P1711: smd-proto-pad, heliopsis-modules:smd-proto-pad, F.Cu at (161.5, 101.6)
- added P1712: smd-proto-pad, heliopsis-modules:smd-proto-pad, F.Cu at (161.5, 102.9)
- added P1713: smd-proto-pad, heliopsis-modules:smd-proto-pad, F.Cu at (161.5, 104.1)
- added P1714: smd-proto-pad, heliopsis-modules:smd-proto-pad, F.Cu at (161.5, 105.4)
- added P1715: smd-proto-pad, heliopsis-modules:smd-proto-pad, F.Cu at (161.5, 106.7)
- added P172: smd-proto-pad, heliopsis-modules:smd-proto-pad, F.Cu at (161.5, 90.2)
- added P173: smd-proto-pad, heliopsis-modules:smd-proto-pad, F.Cu at (161.5, 91.4)
- added P174: smd-proto-pad, heliopsis-modules:smd-proto-pad, F.Cu at (161.5, 92.7)
- added P175: smd-proto-pad, heliopsis-modules:smd-proto-pad, F.Cu at (161.5, 94.0)
- added P176: smd-proto-pad, heliopsis-modules:smd-proto-pad, F.Cu at (161.5, 95.2)
- added P177: smd-proto-pad, heliopsis-modules:smd-proto-pad, F.Cu at (161.5, 96.5)
- added P178: smd-proto-pad, heliopsis-modules:smd-proto-pad, F.Cu at (161.5, 97.8)
- added P179: smd-proto-pad, heliopsis-modules:smd-proto-pad, F.Cu at (161.5, 99.1)
- added P181: smd-proto-pad, heliopsis-modules:smd-proto-pad, F.Cu at (159.9, 88.9)
- added P1810: smd-proto-pad, heliopsis-modules:smd-proto-pad, F.Cu at (159.9, 100.3)
- added P1811: smd-proto-pad, heliopsis-modules:smd-proto-pad, F.Cu at (159.9, 101.6)
- added P1812: smd-proto-pad, heliopsis-modules:smd-proto-pad, F.Cu at (159.9, 102.9)
- added P1813: smd-proto-pad, heliopsis-modules:smd-proto-pad, F.Cu at (159.9, 104.1)
- added P1814: smd-proto-pad, heliopsis-modules:smd-proto-pad, F.Cu at (159.9, 105.4)
- added P1815: smd-proto-pad, heliopsis-modules:smd-proto-pad, F.Cu at (159.9, 106.7)
- added P182: smd-proto-pad, heliopsis-modules:smd-proto-pad, F.Cu at (159.9, 90.2)
- added P183: smd-proto-pad, heliopsis-modules:smd-proto-pad, F.Cu at (159.9, 91.4)
- added P184: smd-proto-pad, heliopsis-modules:smd-proto-pad, F.Cu at (159.9, 92.7)
- added P185: smd-proto-pad, heliopsis-modules:smd-proto-pad, F.Cu at (159.9, 94.0)
- added P186: smd-proto-pad, heliopsis-modules:smd-proto-pad, F.Cu at (159.9, 95.2)
- added P187: smd-proto-pad, heliopsis-modules:smd-proto-pad, F.Cu at (159.9, 96.5)
- added P188: smd-proto-pad, heliopsis-modules:smd-proto-pad, F.Cu at (159.9, 97.8)
- added P189: smd-proto-pad, heliopsis-modules:smd-proto-pad, F.Cu at (159.9, 99.1)
- added P191: smd-proto-pad, heliopsis-modules:smd-proto-pad, F.Cu at (158.2, 88.9)
- added P1910: smd-proto-pad, heliopsis-modules:smd-proto-pad, F.Cu at (158.2, 100.3)
- added P1911: smd-proto-pad, heliopsis-modules:smd-proto-pad, F.Cu at (158.2, 101.6)
- added P1912: smd-proto-pad, heliopsis-modules:smd-proto-pad, F.Cu at (158.2, 102.9)
- added P1913: smd-proto-pad, heliopsis-modules:smd-proto-pad, F.Cu at (158.2, 104.1)
- added P1914: smd-proto-pad, heliopsis-modules:smd-proto-pad, F.Cu at (158.2, 105.4)
- added P1915: smd-proto-pad, heliopsis-modules:smd-proto-pad, F.Cu at (158.2, 106.7)
- added P192: smd-proto-pad, heliopsis-modules:smd-proto-pad, F.Cu at (158.2, 90.2)
- added P193: smd-proto-pad, heliopsis-modules:smd-proto-pad, F.Cu at (158.2, 91.4)
- added P194: smd-proto-pad, heliopsis-modules:smd-proto-pad, F.Cu at (158.2, 92.7)
- added P195: smd-proto-pad, heliopsis-modules:smd-proto-pad, F.Cu at (158.2, 94.0)
- added P196: smd-proto-pad, heliopsis-modules:smd-proto-pad, F.Cu at (158.2, 95.2)
- added P197: smd-proto-pad, heliopsis-modules:smd-proto-pad, F.Cu at (158.2, 96.5)
- added P198: smd-proto-pad, heliopsis-modules:smd-proto-pad, F.Cu at (158.2, 97.8)
- added P199: smd-proto-pad, heliopsis-modules:smd-proto-pad, F.Cu at (158.2, 99.1)
- added PA1: HELIOPSIS-PTH-PROTO-AREA, heliopsis-modules:HELIOPSIS-PTH-PROTO-AREA, F.Cu at (137.2, 96.5)
