File: hardware/heliopsis/heliopsis.kicad_pcb (KiCad board)
At the start: 2 copper layers, 70.7 x 53.3 mm, 311 parts, among them J1 NEIGHBOR1, J11 NEIGHBOR1, J12 NEIGHBOR2, J17 BONUS_ROW, J2 NEIGHBOR2, J7 BONUS_ROW

Commit message: Update date for new version
Other:
- board text added: "29 September 2016"
- board text removed: "2 September 2016"
Changed lines of the file:
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@@
   (gr_line (start 177.9016 92.3544) (end 177.8508 94.0054) (angle 90) (layer Edge.Cuts) (width 0.15))
   (gr_line (start 177.9524 90.5002) (end 177.9016 92.3544) (angle 90) (layer Edge.Cuts) (width 0.15))
-  (gr_text "2 September 2016" (at 153.416 114.681) (layer F.SilkS)
+  (gr_text "29 September 2016" (at 153.416 114.681) (layer F.SilkS)
     (effects (font (size 0.762 0.5715) (thickness 0.1143)))
   )
